Commit message: printf -> print_param

File: realsense_gazebo_description/urdf/_d435.gazebo.xacro (robot description, xacro)
@@ -70,4 +70,5 @@
       <sensor name="${camera_name}ired1" type="camera">
         <camera name="${camera_name}">
+          <pose>0 0 0 ${M_PI} 0 0</pose>
           <horizontal_fov>${85.2*deg_to_rad}</horizontal_fov>
           <image>

File: realsense_gazebo_description/urdf/_d435.urdf.xacro (robot description, xacro)
@@ -18,12 +18,12 @@
                                           enable_pointCloud:=false
                                           clip_distance:=-1.0
-                                          depth_width:=1280
-                                          depth_height:=720
+                                          depth_width:=640
+                                          depth_height:=480
                                           depth_fps:=30
                                           infra_width:=640
                                           infra_height:=480
                                           infra_fps:=30
-                                          color_width:=1920
-                                          color_height:=1080
+                                          color_width:=640
+                                          color_height:=480
                                           color_fps:=30
                                           visualize:=false
@@ -46,4 +46,5 @@
     <xacro:property name="d435_cam_depth_px" value="${d435_cam_mount_from_center_offset}"/>
     <xacro:property name="d435_cam_depth_py" value="0.0175"/>
+    <!-- <xacro:property name="d435_cam_depth_py" value="1.0"/> -->
     <xacro:property name="d435_cam_depth_pz" value="${d435_cam_height/2}"/>
     <material name="${name}_aluminum">
@@ -78,5 +79,5 @@
       <inertial>
         <!-- The following are not reliable values, and should not be used for modeling -->
-        <mass value="1e-5"/>
+        <mass value="0.70"/>
         <origin xyz="0 0 0"/>
         <inertia ixx="1e-10" ixy="0.0" ixz="0.0"

File: realsense_gazebo_description/urdf/_d435i.gazebo.xacro (robot description, xacro)
@@ -88,5 +88,5 @@
             <type>gaussian</type>
             <mean>0.0</mean>
-            <stddev>0.05</stddev>
+            <stddev>0.005</stddev>
           </noise>
         </camera>
